Commit message: adapt configuration for dual arm planning

File: panda_description/urdf/dual_panda.urdf.xacro (robot description, xacro)
@@ -5,6 +5,34 @@
   <xacro:include filename="$(find moveit_resources_panda_description)/urdf/panda_arm.xacro"/>
   <xacro:include filename="$(find moveit_resources_panda_description)/urdf/hand.xacro"/>
+  <link name="world"/>
   <!-- box shaped table as base for the 2 Pandas -->
   <link name="base">
+    <visual>
+      <origin xyz="0.09 0 0.5" rpy="0 0 0" />
+      <geometry>
+        <box size="0.8 1.6 1" />
+      </geometry>
+      <material name="White">
+        <color rgba="1.0 1.0 1.0 1.0" />
+      </material>
+    </visual>
+    <collision>
+      <origin xyz="0.29 0 0.5" rpy="0 0 0" />
+      <geometry>
+        <box size="0.8 1.6 1" />
+      </geometry>
+    </collision>
+    <inertial>
+      <origin xyz="0.0 0.0 0.0" rpy="0.0 0.0 0.0"/>
+      <mass value="10.0"/>
+      <inertia ixx="0.001" ixy="0.0" ixz="0.001" iyy="0.0" iyz="0.0" izz="0.001"/>
+    </inertial>
+  </link>
+  <joint name="base_to_world" type="fixed">
+        <parent link="world"/>
+        <child link="base"/>
+        <origin xyz="0.0 0.0 0.0" rpy="0.0 0.0 0.0"/>
+  </joint>
+  <!-- <link name="base">
     <visual>
       <origin xyz="0 0 0.5" rpy="0 0 0"/>
@@ -22,10 +50,10 @@
       </geometry>
     </collision>
-  </link>
+  </link> -->
   <!-- right arm with gripper -->
-  <xacro:panda_arm arm_id="$(arg arm_id_1)" connected_to="base"  xyz="0 -0.5 1"/>
+  <xacro:panda_arm arm_id="$(arg arm_id_1)" connected_to="base"  xyz="0 -0.281 1"/>
   <xacro:hand ns="$(arg arm_id_1)" rpy="0 0 0" connected_to="$(arg arm_id_1)_link8"/>
   <!-- left arm with gripper -->
-  <xacro:panda_arm arm_id="$(arg arm_id_2)" connected_to="base"  xyz="0 0.5 1"/>
+  <xacro:panda_arm arm_id="$(arg arm_id_2)" connected_to="base"  xyz="0 0.281 1"/>
   <xacro:hand ns="$(arg arm_id_2)" rpy="0 0 0" connected_to="$(arg arm_id_2)_link8"/>
 </robot>

Commit message: task planning milestone

File: panda_description/urdf/dual_panda.urdf.xacro (robot description, xacro)
@@ -18,5 +18,5 @@
     </visual>
     <collision>
-      <origin xyz="0.29 0 0.5" rpy="0 0 0" />
+      <origin xyz="0.09 0 0.5" rpy="0 0 0" />
       <geometry>
         <box size="0.8 1.6 1" />
@@ -52,8 +52,8 @@
   </link> -->
   <!-- right arm with gripper -->
-  <xacro:panda_arm arm_id="$(arg arm_id_1)" connected_to="base"  xyz="0 -0.281 1"/>
+  <xacro:panda_arm arm_id="$(arg arm_id_1)" connected_to="base"  xyz="0 0.281 1"/>
   <xacro:hand ns="$(arg arm_id_1)" rpy="0 0 ${-pi/4}" connected_to="$(arg arm_id_1)_link8"/>
   <!-- left arm with gripper -->
-  <xacro:panda_arm arm_id="$(arg arm_id_2)" connected_to="base"  xyz="0 0.281 1"/>
+  <xacro:panda_arm arm_id="$(arg arm_id_2)" connected_to="base"  xyz="0 -0.281 1"/>
   <xacro:hand ns="$(arg arm_id_2)" rpy="0 0 ${-pi/4}" connected_to="$(arg arm_id_2)_link8"/>
 </robot>

Commit message: Merge branch 'master' of https://github.com/sofiadig/moveit_resources

File: panda_description/urdf/dual_panda.urdf.xacro (robot description, xacro)
@@ -9,10 +9,10 @@
   <link name="base">
     <visual>
-      <origin xyz="0.09 0 0.5" rpy="0 0 0" />
+      <origin xyz="0.29 0 0.5" rpy="0 0 0" />
       <geometry>
-        <box size="0.8 1.6 1" />
+        <box size="1.2 1.6 1" />
       </geometry>
       <material name="White">
-        <color rgba="1.0 1.0 1.0 1.0" />
+        <color rgba="1.0 1.0 1.0 0.7" />
       </material>
     </visual>
